File: NS FPGA V2 iCE/NS FPGA V2 iCE.kicad_pcb (KiCad board)
At the start: 4 copper layers, 27 x 55.5 mm, 68 parts, among them J1 USB_C_Receptacle_USB2.0_14P, J2 Conn_01x20_Pin, J3 Conn_01x20_Pin, J4 Conn_02x03_Odd_Even, J5 Conn_02x03_Odd_Even, J6 Conn_01x07_Pin, SW1 SW_Push, U1 ICE40UP5K-SG48ITR, U2 W25Q128JVS, U3 CP2102N-Axx-xQFN24, U4 AP2112K-3.3, U5 AP2112K-1.2, U6 AP2112K-2.5, U7 AP2112K-1.8, Y1 SG-210STF

Commit message: completed
Parts:
- added G***: LOGO, LOGO, F.Cu at (182.5, 70.0)
Routing:
- net /D+: track 6.24 -> 7.24 mm, vias 0 -> 2
Other:
- board text added: "0a"
- board text added: "12a"
- board text added: "18a"
- board text added: "20a"
- board text added: "22a"
- board text added: "23b"
- board text added: "24a"
- board text added: "29b"
- board text added: "2a"
- board text added: "36b"
- board text added: "37a"
- board text added: "38b"
- board text added: "39a"
- board text added: "3b_G6"
- board text added: "3v3"
- board text added: "41a"
- board text added: "42b"
- board text added: "43a"
- board text added: "44b"
- board text added: "45a_G1"
- board text added: "46b_G0"
- board text added: "48b"
- board text added: "49a"
- board text added: "4a"
- board text added: "50b"
- board text added: "5V"
- board text added: "5b"
- board text added: "6a"
- board text added: "8a"
- board text added: "9b"
- board text added: "CRESET_B"
- board text added: "GND"
- board text added: "SPI_SCK"
- board text added: "SPI_SI"
- board text added: "SPI_SO"
- board text added: "SPI_SS"

Commit message: src
Parts:
- added G***: LOGO, LOGO, B.Cu at (189.6, 91.7)

Commit message: done with BOM/CPL
Parts:
- D3: footprint LED_SMD:LED_Cree-PLCC4_5x5mm_CW -> LED_SMD:LED_RGB_Wuerth-PLCC4_3.2x2.8mm_150141M173100
- moved R14 2.88 mm to (187.0, 98.3)
- moved R12 2.07 mm to (193.2, 98.3)
- moved D3 1.06 mm to (190.1, 98.2)
- moved G*** 0.25 mm to (198.0, 100.2)
Routing:
- net +3V3: track 133.3 -> 143.2 mm, vias 7 -> 8
- net Net-(D3-GK): track 1.77 -> 7.33 mm, vias 0 -> 2
- net Net-(U1A-RGB2): track 25.2 -> 22.8 mm
- net Net-(U1A-RGB0): track 15.1 -> 16.7 mm
- net /SPI_SS: track 50.4 -> 51.2 mm
- net Net-(D3-BK): track 2.12 -> 1.53 mm
- added copper zone on B.Cu, net +3V3
